Commit message: Ongoing : src gazebo

File: src_description/urdf/racecar.urdf (robot description, URDF)
Before this commit: robot racecar, 14 links, 13 joints
Joints:
- joint hokuyo_joint: type fixed -> continuous
- joint imu_joint: type fixed -> continuous
- joint zed_camera_joint: type fixed -> continuous
