Commit message: Ongoing : gazebo setup

File: src_description/urdf/macros.xacro (robot description, xacro)
@@ -92,28 +92,3 @@
   </geometry>
 </xacro:macro>
-<!-- transmission macros -->
-<xacro:macro name="wheel_transmission" params="name">
-  <transmission name="${name}_transmission" type="SimpleTransmission">
-    <type>transmission_interface/SimpleTransmission</type>
-    <joint name="${name}_joint">
-      <hardwareInterface>EffortJointInterface</hardwareInterface>
-    </joint>
-    <actuator name="${name}_motor">
-      <hardwareInterface>EffortJointInterface</hardwareInterface>
-      <mechanicalReduction>1</mechanicalReduction>
-    </actuator>
-  </transmission>
-</xacro:macro>
-<xacro:macro name="steering_hinge_transmission" params="name">
-  <transmission name="${name}_transmission" type="SimpleTransmission">
-    <type>transmission_interface/SimpleTransmission</type>
-    <joint name="${name}_joint">
-      <hardwareInterface>EffortJointInterface</hardwareInterface>
-    </joint>
-    <actuator name="${name}_motor">
-      <hardwareInterface>EffortJointInterface</hardwareInterface>
-      <mechanicalReduction>1</mechanicalReduction>
-    </actuator>
-  </transmission>
-</xacro:macro>
 </robot>

File: src_description/urdf/racecar.urdf.xacro (robot description, xacro)
@@ -2,7 +2,7 @@
 <robot name="racecar" xmlns:xacro="http://www.ros.org/wiki/xacro">
   <xacro:include filename="$(find src_description)/urdf/macros.xacro" />
-  <xacro:include filename="$(find src_description)/urdf/racecar.gazebo" />
   <xacro:include filename="$(find src_description)/urdf/materials.xacro" />
-  <!-- Add chassis and it's inertia link -->
+  <!-- we don't need gazebo file now -->
+  <!-- <xacro:include filename="$(find src_description)/urdf/racecar.gazebo" /> -->
   <link name="base_link" />
   <link name="chassis">
@@ -27,5 +27,4 @@
     <child link="chassis_inertia" />
   </joint>
-  <!-- Add the left rear wheel with its joints and tranmissions -->
   <link name="left_rear_wheel">
     <inertial>
@@ -47,6 +46,4 @@
     <limit effort="10" velocity="100" />
   </joint>
-  <xacro:wheel_transmission name="left_rear_wheel" />
-  <!-- Add the right rear wheel with its joints and tranmissions -->
   <link name="right_rear_wheel">
     <inertial>
@@ -68,6 +65,4 @@
     <limit effort="10" velocity="100" />
   </joint>
-  <xacro:wheel_transmission name="right_rear_wheel" />
-  <!-- Add the left steering hinge with its joints and tranmissions -->
   <link name="left_steering_hinge">
     <inertial>
@@ -86,6 +81,4 @@
     <limit lower="-0.7853" upper="0.7853" effort="10" velocity="100" />
   </joint>
-  <xacro:steering_hinge_transmission name="left_steering_hinge" />
-  <!-- Add the right steering hinge with its joints and tranmissions -->
   <link name="right_steering_hinge">
     <inertial>
@@ -104,6 +97,4 @@
     <limit lower="-0.7853" upper="0.7853" effort="10" velocity="100" />
   </joint>
-  <xacro:steering_hinge_transmission name="right_steering_hinge" />
-  <!-- Add the left front wheel with its joints and tranmissions -->
   <link name="left_front_wheel">
     <inertial>
@@ -125,6 +116,4 @@
     <limit effort="10" velocity="100" />
   </joint>
-  <xacro:wheel_transmission name="left_front_wheel" />
-  <!-- Add the left front wheel with its joints and tranmissions -->
   <link name="right_front_wheel">
     <inertial>
@@ -146,6 +135,4 @@
     <limit effort="10" velocity="100"/>
   </joint>
-  <xacro:wheel_transmission name="right_front_wheel" />
-  <!-- Add Hokuyo laser scanner -->
   <link name="laser">
     <inertial>
@@ -172,5 +159,4 @@
     <axis xyz="0 0 1" />
   </joint>
-  <!-- zed camera -->
   <link name="zed_camera_link">
     <inertial>
@@ -202,5 +188,6 @@
   <!-- zed camera lenses -->
   <!-- It seems these have to have a non-zero mass to have a camera attached? -->
-  <link name="camera_link"><!-- this needs to match the name in zed_wrapper/zed_tf.launch -->
+  <!-- this needs to match the name in zed_wrapper/zed_tf.launch -->
+  <link name="camera_link">
     <inertial>
       <mass value="1e-5" />

Commit message: Update : 바퀴 중심으로 joint 축 변경

File: src_description/urdf/macros.xacro (robot description, xacro)
@@ -10,5 +10,6 @@
 </xacro:macro>
 <xacro:macro name="left_wheels_inertial_params">
-  <origin xyz="0 0 -0.0225" rpy="0 0 0" />
+  <!-- <origin xyz="0 0 -0.0225" rpy="0 0 0" /> -->
+  <origin xyz="0 0 -0.0" rpy="0 0 0" />
   <mass value="0.34055" />
   <inertia ixx="0.00026046" ixy="0"          ixz="0"
@@ -17,5 +18,6 @@
 </xacro:macro>
 <xacro:macro name="right_wheels_inertial_params">
-  <origin xyz="0 0 0.0225" rpy="0 0 0" />
+  <!-- <origin xyz="0 0 0.0225" rpy="0 0 0" /> -->
+  <origin xyz="0 0 0.0" rpy="0 0 0" />
   <mass value="0.34055" />
   <inertia ixx="0.00026046" ixy="0"          ixz="0"
@@ -57,5 +59,6 @@
 </xacro:macro>
 <xacro:macro name="left_front_wheel_geometry">
-  <origin xyz="0 0 0" rpy="0 0 0" />
+  <!-- <origin xyz="0 0 0" rpy="0 0 0" /> -->
+  <origin xyz="0 0 0.0225" rpy="0 0 0" />
   <geometry>
     <mesh filename="package://src_description/meshes/left_front_wheel.STL" />
@@ -63,5 +66,6 @@
 </xacro:macro>
 <xacro:macro name="right_front_wheel_geometry">
-  <origin xyz="0 0 0" rpy="0 0 0" />
+  <!-- <origin xyz="0 0 0" rpy="0 0 0" /> -->
+  <origin xyz="0 0 -0.0225" rpy="0 0 0" />
   <geometry>
     <mesh filename="package://src_description/meshes/right_front_wheel.STL" />

File: src_description/urdf/racecar.urdf.xacro (robot description, xacro)
@@ -75,5 +75,6 @@
   </link>
   <joint name="left_steering_hinge_joint" type="revolute">
-    <origin xyz="0.325 0.1 0" rpy="0 1.5708 0" />
+    <!-- <origin xyz="0.325 0.1 0" rpy="0 1.5708 0" /> -->
+    <origin xyz="0.325 0.1225 0" rpy="0 1.5708 0" />
     <parent link="chassis" />
     <child link="left_steering_hinge" />
@@ -90,6 +91,7 @@
     </visual>
   </link>
-  <joint name="right_steering_hinge_joint" type="continuous">
-    <origin xyz="0.325 -0.1 0" rpy="0 1.5708 0" />
+  <joint name="right_steering_hinge_joint" type="revolute">
+    <!-- <origin xyz="0.325 -0.100 0" rpy="0 1.5708 0" /> -->
+    <origin xyz="0.325 -0.1225 0" rpy="0 1.5708 0" />
     <parent link="chassis" />
     <child link="right_steering_hinge" />
