Commit message: Fix : base_footprint added in urdf / odom

File: src_description/urdf/racecar.urdf.xacro (robot description, xacro)
@@ -5,5 +5,11 @@
   <!-- we don't need gazebo file now -->
   <!-- <xacro:include filename="$(find src_description)/urdf/racecar.gazebo" /> -->
+  <link name="base_footprint" />
   <link name="base_link" />
+  <joint name="base_footprint_joint" type="fixed">
+    <parent link="base_footprint"/>
+    <child link="base_link"/>
+    <origin xyz="0 0 0" rpy="0 0 0"/>
+  </joint>
   <link name="chassis">
     <visual>

File: src_gazebo/urdf/src_ackermann.urdf (robot description, URDF)
Before this commit: robot src_ackermann, 14 links, 13 joints
Links:
- added link base_footprint
Joints:
- added joint base_footprint_joint: type fixed, parent base_footprint, child base_link, origin xyz=0 0 0 rpy=0 0 0

File: src_gazebo/urdf/src_ackermann.urdf.xacro (robot description, xacro)
@@ -5,5 +5,11 @@
   <xacro:include filename="$(find src_gazebo)/urdf/materials.xacro" />
   <!-- Add chassis and it's inertia link -->
+  <link name="base_footprint" />
   <link name="base_link" />
+  <joint name="base_footprint_joint" type="fixed">
+      <parent link="base_footprint"/>
+      <child link="base_link"/>
+      <origin xyz="0 0 0" rpy="0 0 0"/>
+  </joint>
   <link name="chassis">
     <visual>
