Commit message: Ongoing : test_description

File: test_description/urdf/src.urdf.xacro (robot description, xacro)
@@ -71,5 +71,8 @@
   </inertial>
   <visual>
-    <!-- <xacro:right_steering_hinge_geometry /> -->
+    <origin xyz="0 0 0" rpy="0 1.5707 0" />
+    <geometry>
+      <cylinder radius="0.01" length="0.01"/>
+    </geometry>
     <material name="grey" />
   </visual>
@@ -103,9 +106,12 @@
   </inertial>
   <visual>
-    <!-- <xacro:right_steering_hinge_geometry /> -->
+    <origin xyz="0 0 0" rpy="0 0 0" />
+    <geometry>
+      <cylinder radius="0.01" length="0.01"/>
+    </geometry>
     <material name="grey" />
   </visual>
 </link>
-<link name="right_front_wheel_1">
+<!-- <link name="right_front_wheel_1">
   <inertial>
     <origin xyz="0.00900022702540075 -6.154013956760629e-08 -3.3086341972438094e-07" rpy="0 0 0"/>
@@ -126,13 +132,13 @@
     </geometry>
   </collision>
-</link>
+</link> -->
 <link name="laser_1">
   <inertial>
-    <origin xyz="-0.0042590635039571785 -0.37493933888071246 0.3244687193227971" rpy="0 0 0"/>
+    <origin xyz="0 0 0" rpy="0 0 0"/>
     <mass value="0.04195569019892212"/>
     <inertia ixx="2.4e-05" iyy="2.3e-05" izz="3.4e-05" ixy="0.0" iyz="1e-06" ixz="-0.0"/>
   </inertial>
   <visual>
-    <origin xyz="-0.0 -0.188744 0.132256" rpy="0 0 0"/>
+    <origin xyz="0 0 0" rpy="0 0 0"/>
     <geometry>
       <mesh filename="package://test_description/meshes/laser_1.stl" scale="0.001 0.001 0.001"/>
@@ -141,5 +147,5 @@
   </visual>
   <collision>
-    <origin xyz="-0.0 -0.188744 0.132256" rpy="0 0 0"/>
+    <origin xyz="0 0 0" rpy="0 0 0"/>
     <geometry>
       <mesh filename="package://test_description/meshes/laser_1.stl" scale="0.001 0.001 0.001"/>
@@ -152,4 +158,5 @@
   <child link="right_rear_wheel_1"/>
   <axis xyz="-1.0 0.0 0.0"/>
+  <limit effort="10" velocity="100" />
 </joint>
 <joint name="left_rear_wheel_joint" type="continuous">
@@ -158,34 +165,38 @@
   <child link="left_rear_wheel_1"/>
   <axis xyz="-1.0 0.0 0.0"/>
+  <limit effort="10" velocity="100" />
 </joint>
 <joint name="right_front_hinge_joint" type="revolute">
-  <origin xyz="0.083267 -0.22236 0.040754" rpy="0 0 0"/>
+  <origin xyz="0.083267 -0.22236 0.040754" rpy="0 1.5708 0"/>
   <parent link="base_link"/>
   <!-- <child link="right_front_wheel_1"/> -->
   <child link="right_steering_hinge"/>
-  <axis xyz="1.0 -0.0 -0.0"/>
-</joint>
-<joint name="right_front_hinge_joint" type="continuous">
-  <origin xyz="0 0 0" rpy="1.5708 0 0" />
+  <axis xyz="-1.0 -0.0 -0.0"/>
+  <limit lower="-0.7853" upper="0.7853" effort="10" velocity="100" />
+</joint>
+<!-- <joint name="right_front_wheel_joint" type="continuous">
+  <origin xyz="0 0 0" rpy="1.5707 0 0" />
   <parent link="right_steering_hinge"/>
   <child link="right_front_wheel_1"/>
-  <axis xyz="1.0 -0.0 -0.0"/>
-</joint>
+  <axis xyz="0 0 -1"/>
+  <limit effort="10" velocity="100" />
+</joint> -->
 <joint name="left_front_hinge_joint" type="revolute">
   <origin xyz="-0.094233 -0.22236 0.040754" rpy="0 0 0"/>
   <parent link="base_link"/>
-  <!-- <child link="left_front_wheel_1"/> -->
   <child link="left_steering_hinge"/>
   <axis xyz="1.0 -0.0 -0.0"/>
-</joint>
-<joint name="right_front_wheel_joint" type="continuous">
-  <origin xyz="0.083267 -0.22236 0.040754" rpy="0 0 0"/>
+  <limit lower="-0.7853" upper="0.7853" effort="10" velocity="100" />
+</joint>
+<joint name="left_front_wheel_joint" type="continuous">
+  <origin xyz="0 0 0" rpy="1.5707 0 0" />
   <parent link="left_steering_hinge"/>
-  <!-- <child link="right_front_wheel_1"/> -->
   <child link="left_front_wheel_1"/>
   <axis xyz="1.0 -0.0 -0.0"/>
+  <limit effort="10" velocity="100" />
 </joint>
 <joint name="laser_joint" type="fixed">
-  <origin xyz="0.0 0.188744 -0.132256" rpy="0 0 0"/>
+  <!-- <origin xyz="0.0 -0.188744 0.132256" rpy="0 0 0"/> -->
+  <origin xyz="0.0 0.0 0.0" rpy="0 0 0"/>
   <parent link="base_link"/>
   <child link="laser_1"/>
