Commit message: Temporary done : urdf

File: test_description/urdf/src_description.urdf.xacro (robot description, xacro)
@@ -14,5 +14,5 @@
       <origin xyz="0 0 0" rpy="0 0 0"/>
       <geometry>
-        <mesh filename="$(find test_description)/meshes/base_link.stl" scale="0.001 0.001 0.001"/>
+        <mesh filename="package://test_description/meshes/base_link.stl" scale="0.001 0.001 0.001"/>
       </geometry>
       <material name="silver"/>
@@ -21,5 +21,5 @@
       <origin xyz="0 0 0" rpy="0 0 0"/>
       <geometry>
-        <mesh filename="$(find test_description)/meshes/base_link.stl" scale="0.001 0.001 0.001"/>
+        <mesh filename="package://test_description/meshes/base_link.stl" scale="0.001 0.001 0.001"/>
       </geometry>
     </collision>
@@ -39,5 +39,5 @@
       <origin rpy="0 0 0" xyz="-0.0 0.089625 -0.050754"/>
       <geometry>
-        <mesh filename="$(find test_description)/meshes/right_rear_wheel.stl" scale="0.001 0.001 0.001"/>
+        <mesh filename="package://test_description/meshes/right_rear_wheel.stl" scale="0.001 0.001 0.001"/>
       </geometry>
       <material name="silver"/>
@@ -46,5 +46,5 @@
       <origin rpy="0 0 0" xyz="-0.0 0.089625 -0.050754"/>
       <geometry>
-        <mesh filename="$(find test_description)/meshes/right_rear_wheel.stl" scale="0.001 0.001 0.001"/>
+        <mesh filename="package://test_description/meshes/right_rear_wheel.stl" scale="0.001 0.001 0.001"/>
       </geometry>
     </collision>
@@ -66,5 +66,5 @@
       <origin rpy="0 0 0" xyz="-0.0 -0.089625 -0.050754"/>
       <geometry>
-        <mesh filename="$(find test_description)/meshes/left_rear_wheel.stl" scale="0.001 0.001 0.001"/>
+        <mesh filename="package://test_description/meshes/left_rear_wheel.stl" scale="0.001 0.001 0.001"/>
       </geometry>
       <material name="silver"/>
@@ -73,5 +73,5 @@
       <origin rpy="0 0 0" xyz="-0.0 -0.089625 -0.050754"/>
       <geometry>
-        <mesh filename="$(find test_description)/meshes/left_rear_wheel.stl" scale="0.001 0.001 0.001"/>
+        <mesh filename="package://test_description/meshes/left_rear_wheel.stl" scale="0.001 0.001 0.001"/>
       </geometry>
     </collision>
@@ -119,5 +119,5 @@
       <origin rpy="0 0 0" xyz="-0.275 0.08875 -0.050754"/>
       <geometry>
-        <mesh filename="$(find test_description)/meshes/right_front_wheel.stl" scale="0.001 0.001 0.001"/>
+        <mesh filename="package://test_description/meshes/right_front_wheel.stl" scale="0.001 0.001 0.001"/>
       </geometry>
       <material name="silver"/>
@@ -126,5 +126,5 @@
       <origin rpy="0 0 0" xyz="-0.275 0.08875 -0.050754"/>
       <geometry>
-        <mesh filename="$(find test_description)/meshes/right_front_wheel.stl" scale="0.001 0.001 0.001"/>
+        <mesh filename="package://test_description/meshes/right_front_wheel.stl" scale="0.001 0.001 0.001"/>
       </geometry>
     </collision>
@@ -172,5 +172,5 @@
       <origin rpy="0 0 0" xyz="-0.275 -0.08875 -0.050754"/>
       <geometry>
-        <mesh filename="$(find test_description)/meshes/left_front_wheel.stl" scale="0.001 0.001 0.001"/>
+        <mesh filename="package://test_description/meshes/left_front_wheel.stl" scale="0.001 0.001 0.001"/>
       </geometry>
       <material name="silver"/>
@@ -179,5 +179,5 @@
       <origin rpy="0 0 0" xyz="-0.275 -0.08875 -0.050754"/>
       <geometry>
-        <mesh filename="$(find test_description)/meshes/left_front_wheel.stl" scale="0.001 0.001 0.001"/>
+        <mesh filename="package://test_description/meshes/left_front_wheel.stl" scale="0.001 0.001 0.001"/>
       </geometry>
     </collision>
@@ -199,5 +199,5 @@
       <origin rpy="0 0 0" xyz="0.0 0.0 0.0"/>
       <geometry>
-        <mesh filename="$(find test_description)/meshes/laser.stl" scale="0.001 0.001 0.001"/>
+        <mesh filename="package://test_description/meshes/laser.stl" scale="0.001 0.001 0.001"/>
       </geometry>
       <material name="silver"/>
@@ -206,5 +206,5 @@
       <origin rpy="0 0 0" xyz="0.0 0.0 0.0"/>
       <geometry>
-        <mesh filename="$(find test_description)/meshes/laser.stl" scale="0.001 0.001 0.001"/>
+        <mesh filename="package://test_description/meshes/laser.stl" scale="0.001 0.001 0.001"/>
       </geometry>
     </collision>
