Commit message: Ongoing : test_description

File: test_description/urdf/src.urdf (robot description, URDF)
Before this commit: robot src, 7 links, 6 joints
Links:
- removed link laser_1
- removed link left_front_wheel_1
- removed link left_rear_wheel_1
- removed link left_steering_hinge
- removed link right_rear_wheel_1
- removed link right_steering_hinge
- added link base_footprint
- added link left_rear_wheel, mass 0.20069792517970372; collision mesh filename=package://test_description/meshes/left_rear_wheel.stl scale=0.001 0.001 0.001; visual mesh filename=package://test_description/meshes/left_rear_wheel.stl scale=0.001 0.001 0.001
- added link right_rear_wheel, mass 0.20069792517970372; collision mesh filename=package://test_description/meshes/right_rear_wheel.stl scale=0.001 0.001 0.001; visual mesh filename=package://test_description/meshes/right_rear_wheel.stl scale=0.001 0.001 0.001
Joints:
- removed joint laser_joint
- removed joint left_front_hinge_joint
- removed joint left_front_wheel_joint
- removed joint right_front_hinge_joint
- added joint base_footprint_joint: type fixed, parent base_footprint, child base_link, origin xyz=0 0 0 rpy=0 0 0
- joint left_rear_wheel_joint: axis -1.0 0.0 0.0 -> 0.0 1.0 0.0; child left_rear_wheel_1 -> left_rear_wheel; limit effort=10 velocity=100 -> (none); origin xyz=0.084142 0.05264 0.040754 rpy=0 0 0 -> xyz=0.0 0.089625 0.050754 rpy=0 0 0
- joint right_rear_wheel_joint: axis -1.0 0.0 0.0 -> 0.0 1.0 0.0; child right_rear_wheel_1 -> right_rear_wheel; limit effort=10 velocity=100 -> (none); origin xyz=-0.095108 0.05264 0.040754 rpy=0 0 0 -> xyz=0.0 -0.089625 0.050754 rpy=0 0 0

File: test_description/urdf/src.urdf.xacro (robot description, xacro)
@@ -1,204 +1,84 @@
 <?xml version="1.0" ?>
 <robot name="src" xmlns:xacro="http://www.ros.org/wiki/xacro">
-<xacro:include filename="$(find test_description)/urdf/materials.xacro" />
-<xacro:include filename="$(find test_description)/urdf/src.gazebo" />
-<link name="base_link">
-  <inertial>
-    <origin xyz="-0.005482772974599414 -0.02435791820697421 0.08495983966151519" rpy="0 0 0"/>
-    <mass value="31.702953623812817"/>
-    <inertia ixx="0.285557" iyy="0.094192" izz="0.298406" ixy="-0.0" iyz="0.013351" ixz="-0.0"/>
-  </inertial>
-  <visual>
+  <xacro:include filename="$(find test_description)/urdf/materials.xacro" />
+  <xacro:include filename="$(find test_description)/urdf/src.gazebo" />
+  <link name="base_footprint" />
+  <link name="base_link">
+    <inertial>
+      <!-- <origin xyz="-0.005482772974599414 -0.02435791820697421 0.08495983966151519" rpy="0 0 0"/> -->
+      <origin rpy="0 0 0" xyz="0.0769978638261129 -2.8140626253308825e-07 0.09495983966151514"/>
+      <mass value="31.702953623812817"/>
+      <inertia ixx="0.094192" ixy="0.0" ixz="-0.013351" iyy="0.285557" iyz="-0.0" izz="0.298406"/>
+    </inertial>
+    <visual>
+      <origin xyz="0 0 0" rpy="0 0 0"/>
+      <geometry>
+        <mesh filename="package://test_description/meshes/base_link.stl" scale="0.001 0.001 0.001"/>
+      </geometry>
+      <material name="silver"/>
+    </visual>
+    <collision>
+      <origin xyz="0 0 0" rpy="0 0 0"/>
+      <geometry>
+        <mesh filename="package://test_description/meshes/base_link.stl" scale="0.001 0.001 0.001"/>
+      </geometry>
+    </collision>
+  </link>
+  <joint name="base_footprint_joint" type="fixed">
+    <parent link="base_footprint"/>
+    <child link="base_link"/>
     <origin xyz="0 0 0" rpy="0 0 0"/>
-    <geometry>
-      <mesh filename="package://test_description/meshes/base_link.stl" scale="0.001 0.001 0.001"/>
-    </geometry>
-    <material name="silver"/>
-  </visual>
-  <collision>
-    <origin xyz="0 0 0" rpy="0 0 0"/>
-    <geometry>
-      <mesh filename="package://test_description/meshes/base_link.stl" scale="0.001 0.001 0.001"/>
-    </geometry>
-  </collision>
-</link>
-<link name="right_rear_wheel_1">
-  <inertial>
-    <origin xyz="-0.008999772974599085 -6.154013969944527e-08 -3.308634169349456e-07" rpy="0 0 0"/>
-    <mass value="0.20069792517970372"/>
-    <inertia ixx="0.00025" iyy="0.00014" izz="0.00014" ixy="0.0" iyz="0.0" ixz="0.0"/>
-  </inertial>
-  <visual>
-    <origin xyz="0.095108 -0.05264 -0.040754" rpy="0 0 0"/>
-    <geometry>
-      <mesh filename="package://test_description/meshes/right_rear_wheel_1.stl" scale="0.001 0.001 0.001"/>
-    </geometry>
-    <material name="silver"/>
-  </visual>
-  <collision>
-    <origin xyz="0.095108 -0.05264 -0.040754" rpy="0 0 0"/>
-    <geometry>
-      <mesh filename="package://test_description/meshes/right_rear_wheel_1.stl" scale="0.001 0.001 0.001"/>
-    </geometry>
-  </collision>
-</link>
-<link name="left_rear_wheel_1">
-  <inertial>
-    <origin xyz="0.009000227025400986 -6.154013991455098e-08 -3.3086341695576227e-07" rpy="0 0 0"/>
-    <mass value="0.20069792517970372"/>
-    <inertia ixx="0.00025" iyy="0.00014" izz="0.00014" ixy="0.0" iyz="0.0" ixz="0.0"/>
-  </inertial>
-  <visual>
-    <origin xyz="-0.084142 -0.05264 -0.040754" rpy="0 0 0"/>
-    <geometry>
-      <mesh filename="package://test_description/meshes/left_rear_wheel_1.stl" scale="0.001 0.001 0.001"/>
-    </geometry>
-    <material name="silver"/>
-  </visual>
-  <collision>
-    <origin xyz="-0.084142 -0.05264 -0.040754" rpy="0 0 0"/>
-    <geometry>
-      <mesh filename="package://test_description/meshes/left_rear_wheel_1.stl" scale="0.001 0.001 0.001"/>
-    </geometry>
-  </collision>
-</link>
-<link name="left_steering_hinge">
-  <inertial>
-    <!-- <origin xyz="0.00900022702540075 -6.154013956760629e-08 -3.3086341972438094e-07" rpy="0 0 0"/> -->
-    <origin xyz="0 0 0" rpy="0 0 0"/>
-    <mass value="0.20069792517970372"/>
-    <inertia ixx="0.00025" iyy="0.00014" izz="0.00014" ixy="0.0" iyz="0.0" ixz="-0.0"/>
-  </inertial>
-  <visual>
-    <origin xyz="0 0 0" rpy="0 1.5707 0" />
-    <geometry>
-      <cylinder radius="0.01" length="0.01"/>
-    </geometry>
-    <material name="grey" />
-  </visual>
-</link>
-<link name="left_front_wheel_1">
-  <inertial>
-    <origin xyz="-0.008999772974599335 -6.154013934556168e-08 -3.308634166990232e-07" rpy="0 0 0"/>
-    <mass value="0.20069792517970372"/>
-    <inertia ixx="0.00025" iyy="0.00014" izz="0.00014" ixy="0.0" iyz="0.0" ixz="0.0"/>
-  </inertial>
-  <visual>
-    <origin xyz="0.094233 0.22236 -0.040754" rpy="0 0 0"/>
-    <geometry>
-      <mesh filename="package://test_description/meshes/left_front_wheel_1.stl" scale="0.001 0.001 0.001"/>
-    </geometry>
-    <material name="silver"/>
-  </visual>
-  <collision>
-    <origin xyz="0.094233 0.22236 -0.040754" rpy="0 0 0"/>
-    <geometry>
-      <mesh filename="package://test_description/meshes/left_front_wheel_1.stl" scale="0.001 0.001 0.001"/>
-    </geometry>
-  </collision>
-</link>
-<link name="right_steering_hinge">
-  <inertial>
-    <!-- <origin xyz="0.00900022702540075 -6.154013956760629e-08 -3.3086341972438094e-07" rpy="0 0 0"/> -->
-    <origin xyz="0 0 0" rpy="0 0 0"/>
-    <mass value="0.20069792517970372"/>
-    <inertia ixx="0.00025" iyy="0.00014" izz="0.00014" ixy="0.0" iyz="0.0" ixz="-0.0"/>
-  </inertial>
-  <visual>
-    <origin xyz="0 0 0" rpy="0 0 0" />
-    <geometry>
-      <cylinder radius="0.01" length="0.01"/>
-    </geometry>
-    <material name="grey" />
-  </visual>
-</link>
-<!-- <link name="right_front_wheel_1">
-  <inertial>
-    <origin xyz="0.00900022702540075 -6.154013956760629e-08 -3.3086341972438094e-07" rpy="0 0 0"/>
-    <mass value="0.20069792517970372"/>
-    <inertia ixx="0.00025" iyy="0.00014" izz="0.00014" ixy="0.0" iyz="0.0" ixz="-0.0"/>
-  </inertial>
-  <visual>
-    <origin xyz="-0.083267 0.22236 -0.040754" rpy="0 0 0"/>
-    <geometry>
-      <mesh filename="package://test_description/meshes/right_front_wheel_1.stl" scale="0.001 0.001 0.001"/>
-    </geometry>
-    <material name="silver"/>
-  </visual>
-  <collision>
-    <origin xyz="-0.083267 0.22236 -0.040754" rpy="0 0 0"/>
-    <geometry>
-      <mesh filename="package://test_description/meshes/right_front_wheel_1.stl" scale="0.001 0.001 0.001"/>
-    </geometry>
-  </collision>
-</link> -->
-<link name="laser_1">
-  <inertial>
-    <origin xyz="0 0 0" rpy="0 0 0"/>
-    <mass value="0.04195569019892212"/>
-    <inertia ixx="2.4e-05" iyy="2.3e-05" izz="3.4e-05" ixy="0.0" iyz="1e-06" ixz="-0.0"/>
-  </inertial>
-  <visual>
-    <origin xyz="0 0 0" rpy="0 0 0"/>
-    <geometry>
-      <mesh filename="package://test_description/meshes/laser_1.stl" scale="0.001 0.001 0.001"/>
-    </geometry>
-    <material name="silver"/>
-  </visual>
-  <collision>
-    <origin xyz="0 0 0" rpy="0 0 0"/>
-    <geometry>
-      <mesh filename="package://test_description/meshes/laser_1.stl" scale="0.001 0.001 0.001"/>
-    </geometry>
-  </collision>
-</link>
-<joint name="right_rear_wheel_joint" type="continuous">
-  <origin xyz="-0.095108 0.05264 0.040754" rpy="0 0 0"/>
-  <parent link="base_link"/>
-  <child link="right_rear_wheel_1"/>
-  <axis xyz="-1.0 0.0 0.0"/>
-  <limit effort="10" velocity="100" />
-</joint>
-<joint name="left_rear_wheel_joint" type="continuous">
-  <origin xyz="0.084142 0.05264 0.040754" rpy="0 0 0"/>
-  <parent link="base_link"/>
-  <child link="left_rear_wheel_1"/>
-  <axis xyz="-1.0 0.0 0.0"/>
-  <limit effort="10" velocity="100" />
-</joint>
-<joint name="right_front_hinge_joint" type="revolute">
-  <origin xyz="0.083267 -0.22236 0.040754" rpy="0 1.5708 0"/>
-  <parent link="base_link"/>
-  <!-- <child link="right_front_wheel_1"/> -->
-  <child link="right_steering_hinge"/>
-  <axis xyz="-1.0 -0.0 -0.0"/>
-  <limit lower="-0.7853" upper="0.7853" effort="10" velocity="100" />
-</joint>
-<!-- <joint name="right_front_wheel_joint" type="continuous">
-  <origin xyz="0 0 0" rpy="1.5707 0 0" />
-  <parent link="right_steering_hinge"/>
-  <child link="right_front_wheel_1"/>
-  <axis xyz="0 0 -1"/>
-  <limit effort="10" velocity="100" />
-</joint> -->
-<joint name="left_front_hinge_joint" type="revolute">
-  <origin xyz="-0.094233 -0.22236 0.040754" rpy="0 0 0"/>
-  <parent link="base_link"/>
-  <child link="left_steering_hinge"/>
-  <axis xyz="1.0 -0.0 -0.0"/>
-  <limit lower="-0.7853" upper="0.7853" effort="10" velocity="100" />
-</joint>
-<joint name="left_front_wheel_joint" type="continuous">
-  <origin xyz="0 0 0" rpy="1.5707 0 0" />
-  <parent link="left_steering_hinge"/>
-  <child link="left_front_wheel_1"/>
-  <axis xyz="1.0 -0.0 -0.0"/>
-  <limit effort="10" velocity="100" />
-</joint>
-<joint name="laser_joint" type="fixed">
-  <!-- <origin xyz="0.0 -0.188744 0.132256" rpy="0 0 0"/> -->
-  <origin xyz="0.0 0.0 0.0" rpy="0 0 0"/>
-  <parent link="base_link"/>
-  <child link="laser_1"/>
-</joint>
+  </joint>
+  <link name="right_rear_wheel">
+    <inertial>
+      <origin rpy="0 0 0" xyz="7.159278319822104e-09 -0.009000281406262398 -3.3086341685167886e-07"/>
+      <mass value="0.20069792517970372"/>
+      <inertia ixx="0.00014" ixy="0.0" ixz="-0.0" iyy="0.00025" iyz="0.0" izz="0.00014"/>
+    </inertial>
+    <visual>
+      <origin rpy="0 0 0" xyz="-0.0 0.089625 -0.050754"/>
+      <geometry>
+        <mesh filename="package://test_description/meshes/right_rear_wheel.stl" scale="0.001 0.001 0.001"/>
+      </geometry>
+      <material name="silver"/>
+    </visual>
+    <collision>
+      <origin rpy="0 0 0" xyz="-0.0 0.089625 -0.050754"/>
+      <geometry>
+        <mesh filename="package://test_description/meshes/right_rear_wheel.stl" scale="0.001 0.001 0.001"/>
+      </geometry>
+    </collision>
+  </link>
+  <joint name="right_rear_wheel_joint" type="continuous">
+    <origin rpy="0 0 0" xyz="0.0 -0.089625 0.050754"/>
+    <parent link="base_link"/>
+    <child link="right_rear_wheel"/>
+    <axis xyz="0.0 1.0 0.0"/>
+  </joint>
+  <link name="left_rear_wheel">
+    <inertial>
+      <origin rpy="0 0 0" xyz="7.1592785340951474e-09 0.008999718593737882 -3.3086341697657895e-07"/>
+      <mass value="0.20069792517970372"/>
+      <inertia ixx="0.00014" ixy="0.0" ixz="-0.0" iyy="0.00025" iyz="-0.0" izz="0.00014"/>
+    </inertial>
+    <visual>
+      <origin rpy="0 0 0" xyz="-0.0 -0.089625 -0.050754"/>
+      <geometry>
+        <mesh filename="package://test_description/meshes/left_rear_wheel.stl" scale="0.001 0.001 0.001"/>
+      </geometry>
+      <material name="silver"/>
+    </visual>
+    <collision>
+      <origin rpy="0 0 0" xyz="-0.0 -0.089625 -0.050754"/>
+      <geometry>
+        <mesh filename="package://test_description/meshes/left_rear_wheel.stl" scale="0.001 0.001 0.001"/>
+      </geometry>
+    </collision>
+  </link>
+  <joint name="left_rear_wheel_joint" type="continuous">
+    <origin rpy="0 0 0" xyz="0.0 0.089625 0.050754"/>
+    <parent link="base_link"/>
+    <child link="left_rear_wheel"/>
+    <axis xyz="0.0 1.0 0.0"/>
+  </joint>
 </robot>

Commit message: Done : src urdf

File: test_description/urdf/src.urdf (robot description, URDF)
Before this commit: robot src, 4 links, 3 joints
Links:
- added link laser, mass 0.04195569019892212; collision mesh filename=package://test_description/meshes/laser.stl scale=0.001 0.001 0.001; visual mesh filename=package://test_description/meshes/laser.stl scale=0.001 0.001 0.001
- added link left_front_wheel, mass 0.20069792517970372; collision mesh filename=package://test_description/meshes/left_front_wheel.stl scale=0.001 0.001 0.001; visual mesh filename=package://test_description/meshes/left_front_wheel.stl scale=0.001 0.001 0.001
- added link left_steering_hinge, mass 0.0002; visual cylinder length=0.01 radius=0.01
- added link right_front_wheel, mass 0.20069792517970372; collision mesh filename=package://test_description/meshes/right_front_wheel.stl scale=0.001 0.001 0.001; visual mesh filename=package://test_description/meshes/right_front_wheel.stl scale=0.001 0.001 0.001
- added link right_steering_hinge, mass 0.0002; visual cylinder length=0.01 radius=0.01
Joints:
- added joint laser_joint: type fixed, parent base_link, child laser, origin xyz=0 0 0 rpy=0 0 0
- added joint left_front_wheel_joint: type continuous, parent left_steering_hinge, child left_front_wheel, origin xyz=0 0 0 rpy=0 0 0, axis 0.0 1.0 0.0
- added joint left_steering_hinge_joint: type revolute, parent base_link, child left_steering_hinge, origin xyz=0.275 0.08875 0.050754 rpy=0 0 0, axis 0 0 1, limit lower=-0.7853 upper=0.7853 effort=10 velocity=100
- added joint right_front_wheel_joint: type continuous, parent right_steering_hinge, child right_front_wheel, origin xyz=0 0 0 rpy=0 0 0, axis 0.0 1.0 0.0
- added joint right_steering_hinge_joint: type revolute, parent base_link, child right_steering_hinge, origin xyz=0.275 -0.08875 0.050754 rpy=0 0 0, axis 0 0 1, limit lower=-0.7853 upper=0.7853 effort=10 velocity=100

File: test_description/urdf/src.urdf.xacro (robot description, xacro)
@@ -82,3 +82,132 @@
     <axis xyz="0.0 1.0 0.0"/>
   </joint>
+  <link name="right_steering_hinge">
+    <inertial>
+      <origin xyz="0 0 0" rpy="0 0 0" />
+      <mass value="0.0002"/>
+      <inertia ixx="4E-06" ixy="0"          ixz="0"
+                           iyy="4E-06"      iyz="0"
+                                            izz="4E-06" />
+      <geometry>
+        <cylinder radius="0.01" length="0.01"/>
+      </geometry>
+    </inertial>
+    <visual>
+      <origin xyz="0 0 0" rpy="0 0 0" />
+      <geometry>
+        <cylinder radius="0.01" length="0.01"/>
+      </geometry>
+      <material name="grey" />
+    </visual>
+  </link>
+  <joint name="right_steering_hinge_joint" type="revolute">
+    <origin rpy="0 0 0" xyz="0.275 -0.08875 0.050754"/>
+    <parent link="base_link" />
+    <child link="right_steering_hinge" />
+    <axis xyz="0 0 1" />
+    <limit lower="-0.7853" upper="0.7853" effort="10" velocity="100" />
+  </joint>
+  <link name="right_front_wheel">
+    <inertial>
+      <origin rpy="0 0 0" xyz="7.159277781720874e-09 -0.009000281406262675 -3.3086341699045674e-07"/>
+      <mass value="0.20069792517970372"/>
+      <inertia ixx="0.00014" ixy="0.0" ixz="-0.0" iyy="0.00025" iyz="-0.0" izz="0.00014"/>
+    </inertial>
+    <visual>
+      <origin rpy="0 0 0" xyz="-0.275 0.08875 -0.050754"/>
+      <geometry>
+        <mesh filename="package://test_description/meshes/right_front_wheel.stl" scale="0.001 0.001 0.001"/>
+      </geometry>
+      <material name="silver"/>
+    </visual>
+    <collision>
+      <origin rpy="0 0 0" xyz="-0.275 0.08875 -0.050754"/>
+      <geometry>
+        <mesh filename="package://test_description/meshes/right_front_wheel.stl" scale="0.001 0.001 0.001"/>
+      </geometry>
+    </collision>
+  </link>
+  <joint name="right_front_wheel_joint" type="continuous">
+    <origin rpy="0 0 0" xyz="0 0 0"/>
+    <parent link="right_steering_hinge"/>
+    <child link="right_front_wheel"/>
+    <axis xyz="0.0 1.0 0.0"/>
+  </joint>
+  <link name="left_steering_hinge">
+    <inertial>
+      <origin xyz="0 0 0" rpy="0 0 0" />
+      <mass value="0.0002"/>
+      <inertia ixx="4E-06" ixy="0"          ixz="0"
+                           iyy="4E-06"      iyz="0"
+                                            izz="4E-06" />
+      <geometry>
+        <cylinder radius="0.01" length="0.01"/>
+      </geometry>
+    </inertial>
+    <visual>
+      <origin xyz="0 0 0" rpy="0 0 0" />
+      <geometry>
+        <cylinder radius="0.01" length="0.01"/>
+      </geometry>
+      <material name="grey" />
+    </visual>
+  </link>
+  <joint name="left_steering_hinge_joint" type="revolute">
+    <origin rpy="0 0 0" xyz="0.275 0.08875 0.050754"/>
+    <parent link="base_link" />
+    <child link="left_steering_hinge" />
+    <axis xyz="0 0 1" />
+    <limit lower="-0.7853" upper="0.7853" effort="10" velocity="100" />
+  </joint>
+  <link name="left_front_wheel">
+    <inertial>
+      <origin rpy="0 0 0" xyz="7.1592781147877815e-09 0.008999718593737646 -3.30863420112959e-07"/>
+      <mass value="0.20069792517970372"/>
+      <inertia ixx="0.00014" ixy="-0.0" ixz="-0.0" iyy="0.00025" iyz="-0.0" izz="0.00014"/>
+    </inertial>
+    <visual>
+      <origin rpy="0 0 0" xyz="-0.275 -0.08875 -0.050754"/>
+      <geometry>
+        <mesh filename="package://test_description/meshes/left_front_wheel.stl" scale="0.001 0.001 0.001"/>
+      </geometry>
+      <material name="silver"/>
+    </visual>
+    <collision>
+      <origin rpy="0 0 0" xyz="-0.275 -0.08875 -0.050754"/>
+      <geometry>
+        <mesh filename="package://test_description/meshes/left_front_wheel.stl" scale="0.001 0.001 0.001"/>
+      </geometry>
+    </collision>
+  </link>
+  <joint name="left_front_wheel_joint" type="continuous">
+    <origin rpy="0 0 0" xyz="0 0 0"/>
+    <parent link="left_steering_hinge"/>
+    <child link="left_front_wheel"/>
+    <axis xyz="0.0 1.0 0.0"/>
+  </joint>
+  <link name="laser">
+    <inertial>
+      <origin rpy="0 0 0" xyz="0.0 0.0 0.0"/>
+      <mass value="0.04195569019892212"/>
+      <inertia ixx="2.3e-05" ixy="-0.0" ixz="-1e-06" iyy="2.4e-05" iyz="-0.0" izz="3.4e-05"/>
+    </inertial>
+    <visual>
+      <origin rpy="0 0 0" xyz="0.0 0.0 0.0"/>
+      <geometry>
+        <mesh filename="package://test_description/meshes/laser.stl" scale="0.001 0.001 0.001"/>
+      </geometry>
+      <material name="silver"/>
+    </visual>
+    <collision>
+      <origin rpy="0 0 0" xyz="0.0 0.0 0.0"/>
+      <geometry>
+        <mesh filename="package://test_description/meshes/laser.stl" scale="0.001 0.001 0.001"/>
+      </geometry>
+    </collision>
+  </link>
+  <joint name="laser_joint" type="fixed">
+    <origin rpy="0 0 0" xyz="0 0 0"/>
+    <parent link="base_link"/>
+    <child link="laser"/>
+  </joint>
 </robot>

Commit message: Ongoing : src gazebo

File: test_description/urdf/src.urdf (robot description, URDF)
Before this commit: robot src, 9 links, 8 joints
Links:
- link base_link: geometry collision mesh filename=/home/kimsooyoung/ros2_ws/install/test_description/share/te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 scale=0.001 0.001 0.001; visual mesh filename=/home/kimsooyoung/ros2_ws/install/test_description/share/te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 scale=0.001 0.001 0.001
- link laser: geometry collision mesh filename=/home/kimsooyoung/ros2_ws/install/test_description/share/te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 scale=0.001 0.001 0.001; visual mesh filename=/home/kimsooyoung/ros2_ws/install/test_description/share/te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 scale=0.001 0.001 0.001
- link left_front_wheel: geometry collision mesh filename=/home/kimsooyoung/ros2_ws/install/test_description/share/te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 scale=0.001 0.001 0.001; visual mesh filename=/home/kimsooyoung/ros2_ws/install/test_description/share/te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 scale=0.001 0.001 0.001
- link left_rear_wheel: geometry collision mesh filename=/home/kimsooyoung/ros2_ws/install/test_description/share/te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 scale=0.001 0.001 0.001; visual mesh filename=/home/kimsooyoung/ros2_ws/install/test_description/share/te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 scale=0.001 0.001 0.001
- link left_steering_hinge: mass 0.0002 -> 0.100
- link right_front_wheel: geometry collision mesh filename=/home/kimsooyoung/ros2_ws/install/test_description/share/te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 scale=0.001 0.001 0.001; visual mesh filename=/home/kimsooyoung/ros2_ws/install/test_description/share/te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 scale=0.001 0.001 0.001
- link right_rear_wheel: geometry collision mesh filename=/home/kimsooyoung/ros2_ws/install/test_description/share/te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 scale=0.001 0.001 0.001; visual mesh filename=/home/kimsooyoung/ros2_ws/install/test_description/share/te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 scale=0.001 0.001 0.001
- link right_steering_hinge: mass 0.0002 -> 0.100
Joints:
- joint left_front_wheel_joint: limit (none) -> effort=10 velocity=100
- joint left_rear_wheel_joint: limit (none) -> effort=10 velocity=100
- joint left_steering_hinge_joint: limit lower=-0.7853 upper=0.7853 effort=10 velocity=100 -> lower=-1.0 upper=1.0 effort=10 velocity=100
- joint right_front_wheel_joint: limit (none) -> effort=10 velocity=100
- joint right_rear_wheel_joint: limit (none) -> effort=10 velocity=100
