Commit message: Forgive : test description 보류!

File: test_description/urdf/src.urdf (robot description, URDF)
Before this commit: robot src, 9 links, 8 joints
Links:
- link left_steering_hinge: geometry visual mesh filename=/home/kimsooyoung/ros2_ws/install/test_description/share/te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
- link right_steering_hinge: geometry visual mesh filename=/home/kimsooyoung/ros2_ws/install/test_description/share/te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
Joints:
- joint left_front_wheel_joint: origin xyz=0 0 0 rpy=0 0 0 -> xyz=0 0 0 rpy=0 1.5707 0
- joint right_front_wheel_joint: origin xyz=0 0 0 rpy=0 0 0 -> xyz=0 0 0 rpy=0 1.5707 0

File: test_description/urdf/src.urdf.xacro (robot description, xacro)
@@ -91,12 +91,9 @@
                            iyy="4E-06"      iyz="0"
                                             izz="4E-06" />
-      <geometry>
-        <cylinder radius="0.01" length="0.01"/>
-      </geometry>
-    </inertial>
-    <visual>
-      <origin xyz="0 0 0" rpy="0 0 0" />
-      <geometry>
-        <cylinder radius="0.01" length="0.01"/>
+    </inertial>
+    <visual>
+      <origin xyz="0 0 0" rpy="0 0 0" />
+      <geometry>
+        <mesh filename="$(find test_description)/meshes/left_steering_hinge.STL" />
       </geometry>
       <material name="grey" />
@@ -131,5 +128,5 @@
   </link>
   <joint name="right_front_wheel_joint" type="continuous">
-    <origin rpy="0 0 0" xyz="0 0 0"/>
+    <origin rpy="0 1.5707 0" xyz="0 0 0"/>
     <parent link="right_steering_hinge"/>
     <child link="right_front_wheel"/>
@@ -144,12 +141,9 @@
                            iyy="4E-06"      iyz="0"
                                             izz="4E-06" />
-      <geometry>
-        <cylinder radius="0.01" length="0.01"/>
-      </geometry>
-    </inertial>
-    <visual>
-      <origin xyz="0 0 0" rpy="0 0 0" />
-      <geometry>
-        <cylinder radius="0.01" length="0.01"/>
+    </inertial>
+    <visual>
+      <origin xyz="0 0 0" rpy="0 0 0" />
+      <geometry>
+        <mesh filename="$(find test_description)/meshes/left_steering_hinge.STL" />
       </geometry>
       <material name="grey" />
@@ -184,5 +178,5 @@
   </link>
   <joint name="left_front_wheel_joint" type="continuous">
-    <origin rpy="0 0 0" xyz="0 0 0"/>
+    <origin rpy="0 1.5707 0" xyz="0 0 0"/>
     <parent link="left_steering_hinge"/>
     <child link="left_front_wheel"/>

File: test_description/urdf/src_description.urdf.xacro (robot description, xacro)
@@ -131,5 +131,5 @@
   </link>
   <joint name="right_front_wheel_joint" type="continuous">
-    <origin rpy="0 0 0" xyz="0 0 0"/>
+    <origin rpy="0 1.5707 0" xyz="0 0 0"/>
     <parent link="right_steering_hinge"/>
     <child link="right_front_wheel"/>
@@ -184,5 +184,5 @@
   </link>
   <joint name="left_front_wheel_joint" type="continuous">
-    <origin rpy="0 0 0" xyz="0 0 0"/>
+    <origin rpy="0 1.5707 0" xyz="0 0 0"/>
     <parent link="left_steering_hinge"/>
     <child link="left_front_wheel"/>
