Commit message: Fix : hinge joint

File: src_gazebo/urdf/src_ackermann.urdf (robot description, URDF)
Before this commit: robot src_ackermann, 15 links, 14 joints
Joints:
- joint right_steering_hinge_joint: type continuous -> revolute

File: src_gazebo/urdf/src_ackermann.urdf.xacro (robot description, xacro)
@@ -98,5 +98,5 @@
     </visual>
   </link>
-  <joint name="right_steering_hinge_joint" type="continuous">
+  <joint name="right_steering_hinge_joint" type="revolute">
     <!-- <origin xyz="0.325 -0.100 0" rpy="0 1.5708 0" /> -->
     <origin xyz="0.325 -0.1225 0" rpy="0 1.5708 0" />
