Commit message: Ongoing : src gazebo

File: src_gazebo/urdf/macros.xacro (robot description, xacro)
@@ -1,119 +1,84 @@
 <?xml version="1.0"?>
-<robot name="racecar" xmlns:xacro="http://www.ros.org/wiki/xacro">
-<!-- inertial parameter macros -->
-<xacro:macro name="chassis_inertial_params">
-  <origin xyz="0.1477 0 0" rpy="0 0 0" />
-  <mass value="4.0" />
-  <inertia ixx="0.010609" ixy="0"          ixz="0"
-                          iyy="0.050409"   iyz="0"
-                                           izz="0.05865" />
-</xacro:macro>
-<xacro:macro name="left_wheels_inertial_params">
-  <origin xyz="0 0 -0.0225" rpy="0 0 0" />
-  <mass value="0.34055" />
-  <inertia ixx="0.00026046" ixy="0"          ixz="0"
-                            iyy="0.00026046" iyz="0"
-                                             izz="0.00041226" />
-</xacro:macro>
-<xacro:macro name="right_wheels_inertial_params">
-  <origin xyz="0 0 0.0225" rpy="0 0 0" />
-  <mass value="0.34055" />
-  <inertia ixx="0.00026046" ixy="0"          ixz="0"
-                            iyy="0.00026046" iyz="0"
-                                             izz="0.00041226" />
-</xacro:macro>
-<xacro:macro name="steering_hinge_inertial_params">
-  <origin xyz="0 0 0" rpy="0 0 0" />
-  <mass value="0.100" />
-  <inertia ixx="4E-06" ixy="0"           ixz="0"
-                            iyy="4E-06"  iyz="0"
-                                              izz="4E-06" />
-</xacro:macro>
-<xacro:macro name="hokuyo_inertial_params">
-  <origin xyz="0 0 0" rpy="0 0 0" />
-  <mass value="0.130" />
-  <inertia ixx="4E-06" ixy="0"           ixz="0"
-                            iyy="4E-06"  iyz="0"
-                                              izz="4E-06" />
-</xacro:macro>
-<!-- geometry macros -->
-<xacro:macro name="chassis_geometry">
-  <origin xyz="0 0 0" rpy="0 0 0" />
-  <geometry>
-    <mesh filename="$(find sw_ros2_control_gazebo)/meshes/chassis.STL" />
-  </geometry>
-</xacro:macro>
-<xacro:macro name="left_rear_wheel_geometry">
-  <origin xyz="0 0 0" rpy="0 0 0" />
-  <geometry>
-    <mesh filename="$(find sw_ros2_control_gazebo)/meshes/left_rear_wheel.STL" />
-  </geometry>
-</xacro:macro>
-<xacro:macro name="right_rear_wheel_geometry">
-  <origin xyz="0 0 0" rpy="0 0 0" />
-  <geometry>
-    <mesh filename="$(find sw_ros2_control_gazebo)/meshes/right_rear_wheel.STL" />
-  </geometry>
-</xacro:macro>
-<xacro:macro name="left_front_wheel_geometry">
-  <origin xyz="0 0 0" rpy="0 0 0" />
-  <geometry>
-    <mesh filename="$(find sw_ros2_control_gazebo)/meshes/left_front_wheel.STL" />
-  </geometry>
-</xacro:macro>
-<xacro:macro name="right_front_wheel_geometry">
-  <origin xyz="0 0 0" rpy="0 0 0" />
-  <geometry>
-    <mesh filename="$(find sw_ros2_control_gazebo)/meshes/right_front_wheel.STL" />
-  </geometry>
-</xacro:macro>
-<xacro:macro name="left_steering_hinge_geometry">
-  <origin xyz="0 0 0" rpy="0 0 0" />
-  <geometry>
-    <mesh filename="$(find sw_ros2_control_gazebo)/meshes/left_steering_hinge.STL" />
-  </geometry>
-</xacro:macro>
-<xacro:macro name="right_steering_hinge_geometry">
-  <origin xyz="0 0 0" rpy="0 0 0" />
-  <geometry>
-    <mesh filename="$(find sw_ros2_control_gazebo)/meshes/right_steering_hinge.STL" />
-  </geometry>
-</xacro:macro>
-<xacro:macro name="left_wheels_collision_geometry">
-  <origin xyz="0 0 -0.0225" rpy="0 0 0" />
-  <geometry>
-    <cylinder length="0.045" radius="0.05" />
-  </geometry>
-</xacro:macro>
-<xacro:macro name="right_wheels_collision_geometry">
-  <origin xyz="0 0 0.0225" rpy="0 0 0" />
-  <geometry>
-    <cylinder length="0.045" radius="0.05" />
-  </geometry>
-</xacro:macro>
-<!-- transmission macros -->
-<xacro:macro name="wheel_transmission" params="name">
-  <transmission name="${name}_transmission" type="SimpleTransmission">
-    <type>transmission_interface/SimpleTransmission</type>
-    <joint name="${name}_joint">
-      <hardwareInterface>EffortJointInterface</hardwareInterface>
-    </joint>
-    <actuator name="${name}_motor">
-      <hardwareInterface>EffortJointInterface</hardwareInterface>
-      <mechanicalReduction>1</mechanicalReduction>
-    </actuator>
-  </transmission>
-</xacro:macro>
-<xacro:macro name="steering_hinge_transmission" params="name">
-  <transmission name="${name}_transmission" type="SimpleTransmission">
-    <type>transmission_interface/SimpleTransmission</type>
-    <joint name="${name}_joint">
-      <hardwareInterface>EffortJointInterface</hardwareInterface>
-    </joint>
-    <actuator name="${name}_motor">
-      <hardwareInterface>EffortJointInterface</hardwareInterface>
-      <mechanicalReduction>1</mechanicalReduction>
-    </actuator>
-  </transmission>
-</xacro:macro>
+<robot name="src_ackermann" xmlns:xacro="http://www.ros.org/wiki/xacro">
+  <!-- inertial parameter macros -->
+  <xacro:macro name="chassis_inertial_params">
+    <origin xyz="0.1477 0 0" rpy="0 0 0" />
+    <mass value="4.0" />
+    <inertia ixx="0.010609" ixy="0" ixz="0" iyy="0.050409" iyz="0" izz="0.05865" />
+  </xacro:macro>
+  <xacro:macro name="left_wheels_inertial_params">
+    <origin xyz="0 0 -0.0225" rpy="0 0 0" />
+    <mass value="0.34055" />
+    <inertia ixx="0.00026046" ixy="0" ixz="0" iyy="0.00026046" iyz="0" izz="0.00041226" />
+  </xacro:macro>
+  <xacro:macro name="right_wheels_inertial_params">
+    <origin xyz="0 0 0.0225" rpy="0 0 0" />
+    <mass value="0.34055" />
+    <inertia ixx="0.00026046" ixy="0" ixz="0" iyy="0.00026046" iyz="0" izz="0.00041226" />
+  </xacro:macro>
+  <xacro:macro name="steering_hinge_inertial_params">
+    <origin xyz="0 0 0" rpy="0 0 0" />
+    <mass value="0.100" />
+    <inertia ixx="4E-06" ixy="0" ixz="0" iyy="4E-06" iyz="0" izz="4E-06" />
+  </xacro:macro>
+  <xacro:macro name="hokuyo_inertial_params">
+    <origin xyz="0 0 0" rpy="0 0 0" />
+    <mass value="0.130" />
+    <inertia ixx="4E-06" ixy="0" ixz="0" iyy="4E-06" iyz="0" izz="4E-06" />
+  </xacro:macro>
+  <!-- geometry macros -->
+  <xacro:macro name="chassis_geometry">
+    <origin xyz="0 0 0" rpy="0 0 0" />
+    <geometry>
+      <mesh filename="$(find sw_ros2_control_gazebo)/meshes/chassis.STL" />
+    </geometry>
+  </xacro:macro>
+  <xacro:macro name="left_rear_wheel_geometry">
+    <origin xyz="0 0 0" rpy="0 0 0" />
+    <geometry>
+      <mesh filename="$(find sw_ros2_control_gazebo)/meshes/left_rear_wheel.STL" />
+    </geometry>
+  </xacro:macro>
+  <xacro:macro name="right_rear_wheel_geometry">
+    <origin xyz="0 0 0" rpy="0 0 0" />
+    <geometry>
+      <mesh filename="$(find sw_ros2_control_gazebo)/meshes/right_rear_wheel.STL" />
+    </geometry>
+  </xacro:macro>
+  <xacro:macro name="left_front_wheel_geometry">
+    <origin xyz="0 0 0" rpy="0 0 0" />
+    <geometry>
+      <mesh filename="$(find sw_ros2_control_gazebo)/meshes/left_front_wheel.STL" />
+    </geometry>
+  </xacro:macro>
+  <xacro:macro name="right_front_wheel_geometry">
+    <origin xyz="0 0 0" rpy="0 0 0" />
+    <geometry>
+      <mesh filename="$(find sw_ros2_control_gazebo)/meshes/right_front_wheel.STL" />
+    </geometry>
+  </xacro:macro>
+  <xacro:macro name="left_steering_hinge_geometry">
+    <origin xyz="0 0 0" rpy="0 0 0" />
+    <geometry>
+      <mesh filename="$(find sw_ros2_control_gazebo)/meshes/left_steering_hinge.STL" />
+    </geometry>
+  </xacro:macro>
+  <xacro:macro name="right_steering_hinge_geometry">
+    <origin xyz="0 0 0" rpy="0 0 0" />
+    <geometry>
+      <mesh filename="$(find sw_ros2_control_gazebo)/meshes/right_steering_hinge.STL" />
+    </geometry>
+  </xacro:macro>
+  <xacro:macro name="left_wheels_collision_geometry">
+    <origin xyz="0 0 -0.0225" rpy="0 0 0" />
+    <geometry>
+      <cylinder length="0.045" radius="0.05" />
+    </geometry>
+  </xacro:macro>
+  <xacro:macro name="right_wheels_collision_geometry">
+    <origin xyz="0 0 0.0225" rpy="0 0 0" />
+    <geometry>
+      <cylinder length="0.045" radius="0.05" />
+    </geometry>
+  </xacro:macro>
 </robot>

File: src_gazebo/urdf/materials.xacro (robot description, xacro)
@@ -1,27 +1,27 @@
 <?xml version="1.0"?>
-<robot name="racecar" xmlns:xacro="http://www.ros.org/wiki/xacro">
-<material name="black">
-  <color rgba="0.0 0.0 0.0 1.0"/>
-</material>
-<material name="blue">
-  <color rgba="0.0 0.0 0.8 1.0"/>
-</material>
-<material name="green">
-  <color rgba="0.0 0.8 0.0 1.0"/>
-</material>
-<material name="grey">
-  <color rgba="0.2 0.2 0.2 1.0"/>
-</material>
-<material name="orange">
-  <color rgba="${255/255} ${108/255} ${10/255} 1.0"/>
-</material>
-<material name="brown">
-  <color rgba="${222/255} ${207/255} ${195/255} 1.0"/>
-</material>
-<material name="red">
-  <color rgba="0.8 0.0 0.0 1.0"/>
-</material>
-<material name="white">
-  <color rgba="1.0 1.0 1.0 1.0"/>
-</material>
+<robot name="src_ackermann" xmlns:xacro="http://www.ros.org/wiki/xacro">
+  <material name="black">
+    <color rgba="0.0 0.0 0.0 1.0" />
+  </material>
+  <material name="blue">
+    <color rgba="0.0 0.0 0.8 1.0" />
+  </material>
+  <material name="green">
+    <color rgba="0.0 0.8 0.0 1.0" />
+  </material>
+  <material name="grey">
+    <color rgba="0.2 0.2 0.2 1.0" />
+  </material>
+  <material name="orange">
+    <color rgba="${255/255} ${108/255} ${10/255} 1.0" />
+  </material>
+  <material name="brown">
+    <color rgba="${222/255} ${207/255} ${195/255} 1.0" />
+  </material>
+  <material name="red">
+    <color rgba="0.8 0.0 0.0 1.0" />
+  </material>
+  <material name="white">
+    <color rgba="1.0 1.0 1.0 1.0" />
+  </material>
 </robot>

File: src_gazebo/urdf/src_ackermann.urdf (robot description, URDF)
Before this commit: robot racecar, 14 links, 13 joints
Links:
- link laser: geometry collision box size=0.1 0.1 0.1; visual mesh filename=/home/kimsooyoung/ros2_ws/install/src_gazebo/share/src_gaze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

File: src_gazebo/urdf/src_ackermann.urdf.xacro (robot description, xacro)
@@ -1,12 +1,12 @@
 <?xml version="1.0"?>
-<robot name="racecar" xmlns:xacro="http://www.ros.org/wiki/xacro">
-  <xacro:include filename="$(find sw_ros2_control_gazebo)/urdf/clean_racecar/macros.xacro" />
-  <xacro:include filename="$(find sw_ros2_control_gazebo)/urdf/clean_racecar/clean_racecar.gazebo" />
-  <xacro:include filename="$(find sw_ros2_control_gazebo)/urdf/clean_racecar/materials.xacro" />
+<robot name="src_ackermann" xmlns:xacro="http://www.ros.org/wiki/xacro">
+  <xacro:include filename="$(find src_gazebo)/urdf/macros.xacro" />
+  <xacro:include filename="$(find src_gazebo)/urdf/src_ackermann.gazebo" />
+  <xacro:include filename="$(find src_gazebo)/urdf/materials.xacro" />
   <!-- Add chassis and it's inertia link -->
   <link name="base_link" />
   <link name="chassis">
     <visual>
-      <xacro:chassis_geometry/>
+      <xacro:chassis_geometry />
       <material name="blue" />
     </visual>
@@ -47,6 +47,4 @@
     <limit effort="10" velocity="100" />
   </joint>
-  <xacro:wheel_transmission name="left_rear_wheel" />
-  <!-- Add the right rear wheel with its joints and tranmissions -->
   <link name="right_rear_wheel">
     <inertial>
@@ -68,6 +66,4 @@
     <limit effort="10" velocity="100" />
   </joint>
-  <xacro:wheel_transmission name="right_rear_wheel" />
-  <!-- Add the left steering hinge with its joints and tranmissions -->
   <link name="left_steering_hinge">
     <inertial>
@@ -86,6 +82,4 @@
     <limit lower="-1.0" upper="1.0" effort="10" velocity="100" />
   </joint>
-  <xacro:steering_hinge_transmission name="left_steering_hinge" />
-  <!-- Add the right steering hinge with its joints and tranmissions -->
   <link name="right_steering_hinge">
     <inertial>
@@ -104,6 +98,4 @@
     <limit lower="-1.0" upper="1.0" effort="10" velocity="100" />
   </joint>
-  <xacro:steering_hinge_transmission name="right_steering_hinge" />
-  <!-- Add the left front wheel with its joints and tranmissions -->
   <link name="left_front_wheel">
     <inertial>
@@ -125,6 +117,4 @@
     <limit effort="10" velocity="100" />
   </joint>
-  <xacro:wheel_transmission name="left_front_wheel" />
-  <!-- Add the left front wheel with its joints and tranmissions -->
   <link name="right_front_wheel">
     <inertial>
@@ -144,8 +134,6 @@
     <child link="right_front_wheel" />
     <axis xyz="0 0 -1" />
-    <limit effort="10" velocity="100"/>
-  </joint>
-  <xacro:wheel_transmission name="right_front_wheel" />
-  <!-- Add Hokuyo laser scanner -->
+    <limit effort="10" velocity="100" />
+  </joint>
   <link name="laser">
     <inertial>
@@ -153,13 +141,13 @@
     </inertial>
     <collision>
-      <origin xyz="0 0 0" rpy="0 0 0"/>
-      <geometry>
-        <box size="0.1 0.1 0.1"/>
-      </geometry>
-    </collision>
-    <visual>
-      <origin xyz="0 0 0" rpy="0 0 0"/>
-      <geometry>
-        <mesh filename="$(find sw_ros2_control_gazebo)/meshes/hokuyo.dae"/>
+      <origin xyz="0 0 0" rpy="0 0 0" />
+      <geometry>
+        <box size="0.1 0.1 0.1" />
+      </geometry>
+    </collision>
+    <visual>
+      <origin xyz="0 0 0" rpy="0 0 0" />
+      <geometry>
+        <mesh filename="$(find src_gazebo)/meshes/hokuyo.dae" />
         <material name="grey" />
       </geometry>
@@ -167,5 +155,5 @@
   </link>
   <joint name="hokuyo_joint" type="fixed">
-    <origin xyz="0.265 0.0 0.075" rpy="0 0 0"/>
+    <origin xyz="0.265 0.0 0.075" rpy="0 0 0" />
     <parent link="chassis" />
     <child link="laser" />
@@ -176,25 +164,25 @@
     <inertial>
       <mass value="1e-5" />
-      <origin xyz="0 0 0" rpy="0 0 0"/>
+      <origin xyz="0 0 0" rpy="0 0 0" />
       <inertia ixx="1e-6" ixy="0" ixz="0" iyy="1e-6" iyz="0" izz="1e-6" />
     </inertial>
     <collision>
-      <origin xyz="0 0 0" rpy="0 0 0"/>
-      <geometry>
-        <box size="0.033 0.175 0.030"/>
-      </geometry>
-    </collision>
-    <visual>
-      <origin xyz="0 0 0" rpy="0 0 0"/>
-      <geometry>
-        <box size="0.033 0.175 0.030"/>
-      </geometry>
-      <material name="red"/>
+      <origin xyz="0 0 0" rpy="0 0 0" />
+      <geometry>
+        <box size="0.033 0.175 0.030" />
+      </geometry>
+    </collision>
+    <visual>
+      <origin xyz="0 0 0" rpy="0 0 0" />
+      <geometry>
+        <box size="0.033 0.175 0.030" />
+      </geometry>
+      <material name="red" />
     </visual>
   </link>
   <joint name="zed_camera_joint" type="fixed">
-    <origin xyz="0.390 0 0.04" rpy="0 0 0"/>
-    <parent link="chassis"/>
-    <child link="zed_camera_link"/>
+    <origin xyz="0.390 0 0.04" rpy="0 0 0" />
+    <parent link="chassis" />
+    <child link="zed_camera_link" />
     <axis xyz="0 0 1" />
     <!-- <limit lower="0.0" upper="0.0" effort="0.0" velocity="0.0" /> -->
@@ -202,8 +190,9 @@
   <!-- zed camera lenses -->
   <!-- It seems these have to have a non-zero mass to have a camera attached? -->
-  <link name="camera_link"><!-- this needs to match the name in zed_wrapper/zed_tf.launch -->
+  <link name="camera_link">
+    <!-- this needs to match the name in zed_wrapper/zed_tf.launch -->
     <inertial>
       <mass value="1e-5" />
-      <origin xyz="0 0 0" rpy="0 0 0"/>
+      <origin xyz="0 0 0" rpy="0 0 0" />
       <inertia ixx="1e-6" ixy="0" ixz="0" iyy="1e-6" iyz="0" izz="1e-6" />
     </inertial>
@@ -212,30 +201,30 @@
     <inertial>
       <mass value="1e-5" />
-      <origin xyz="0 0 0" rpy="0 0 0"/>
+      <origin xyz="0 0 0" rpy="0 0 0" />
       <inertia ixx="1e-6" ixy="0" ixz="0" iyy="1e-6" iyz="0" izz="1e-6" />
     </inertial>
   </link>
   <joint name="zed_camera_left_joint" type="fixed">
-    <origin xyz="0 0.06 0" rpy="0 0 0"/>
-    <parent link="zed_camera_link"/>
-    <child link="camera_link"/>
+    <origin xyz="0 0.06 0" rpy="0 0 0" />
+    <parent link="zed_camera_link" />
+    <child link="camera_link" />
     <axis xyz="0 0 1" />
   </joint>
   <joint name="zed_camera_right_joint" type="fixed">
-    <origin xyz="0 -0.06 0" rpy="0 0 0"/>
-    <parent link="zed_camera_link"/>
-    <child link="zed_camera_right_link"/>
+    <origin xyz="0 -0.06 0" rpy="0 0 0" />
+    <parent link="zed_camera_link" />
+    <child link="zed_camera_right_link" />
     <axis xyz="0 0 1" />
   </joint>
   <link name="imu_link">
     <inertial>
-      <mass value="0.01"/>
-      <inertia ixx="1.0" ixy="0" ixz="0" iyy="1.0" iyz="0" izz="1.0"/>
+      <mass value="0.01" />
+      <inertia ixx="1.0" ixy="0" ixz="0" iyy="1.0" iyz="0" izz="1.0" />
     </inertial>
   </link>
   <joint name="imu_joint" type="fixed">
-    <origin xyz="0.01 0 0" rpy="0 0 0"/>
-    <parent link="zed_camera_link"/>
-    <child link="imu_link"/>
+    <origin xyz="0.01 0 0" rpy="0 0 0" />
+    <parent link="zed_camera_link" />
+    <child link="imu_link" />
     <!-- <axis xyz="0 0 1" /> -->
   </joint>

Commit message: Update : steering wheel joint updated

File: src_gazebo/urdf/macros.xacro (robot description, xacro)
@@ -8,10 +8,12 @@
   </xacro:macro>
   <xacro:macro name="left_wheels_inertial_params">
-    <origin xyz="0 0 -0.0225" rpy="0 0 0" />
+    <!-- <origin xyz="0 0 -0.0225" rpy="0 0 0" /> -->
+    <origin xyz="0 0 -0.0" rpy="0 0 0" />
     <mass value="0.34055" />
     <inertia ixx="0.00026046" ixy="0" ixz="0" iyy="0.00026046" iyz="0" izz="0.00041226" />
   </xacro:macro>
   <xacro:macro name="right_wheels_inertial_params">
-    <origin xyz="0 0 0.0225" rpy="0 0 0" />
+    <!-- <origin xyz="0 0 0.0225" rpy="0 0 0" /> -->
+    <origin xyz="0 0 0.0" rpy="0 0 0" />
     <mass value="0.34055" />
     <inertia ixx="0.00026046" ixy="0" ixz="0" iyy="0.00026046" iyz="0" izz="0.00041226" />
@@ -31,5 +33,5 @@
     <origin xyz="0 0 0" rpy="0 0 0" />
     <geometry>
-      <mesh filename="$(find sw_ros2_control_gazebo)/meshes/chassis.STL" />
+      <mesh filename="$(find src_gazebo)/meshes/chassis.STL" />
     </geometry>
   </xacro:macro>
@@ -37,5 +39,5 @@
     <origin xyz="0 0 0" rpy="0 0 0" />
     <geometry>
-      <mesh filename="$(find sw_ros2_control_gazebo)/meshes/left_rear_wheel.STL" />
+      <mesh filename="$(find src_gazebo)/meshes/left_rear_wheel.STL" />
     </geometry>
   </xacro:macro>
@@ -43,17 +45,19 @@
     <origin xyz="0 0 0" rpy="0 0 0" />
     <geometry>
-      <mesh filename="$(find sw_ros2_control_gazebo)/meshes/right_rear_wheel.STL" />
+      <mesh filename="$(find src_gazebo)/meshes/right_rear_wheel.STL" />
     </geometry>
   </xacro:macro>
   <xacro:macro name="left_front_wheel_geometry">
-    <origin xyz="0 0 0" rpy="0 0 0" />
+    <!-- <origin xyz="0 0 0" rpy="0 0 0" /> -->
+    <origin xyz="0 0 0.0225" rpy="0 0 0" />
     <geometry>
-      <mesh filename="$(find sw_ros2_control_gazebo)/meshes/left_front_wheel.STL" />
+      <mesh filename="$(find src_gazebo)/meshes/left_front_wheel.STL" />
     </geometry>
   </xacro:macro>
   <xacro:macro name="right_front_wheel_geometry">
-    <origin xyz="0 0 0" rpy="0 0 0" />
+    <!-- <origin xyz="0 0 0" rpy="0 0 0" /> -->
+    <origin xyz="0 0 -0.0225" rpy="0 0 0" />
     <geometry>
-      <mesh filename="$(find sw_ros2_control_gazebo)/meshes/right_front_wheel.STL" />
+      <mesh filename="$(find src_gazebo)/meshes/right_front_wheel.STL" />
     </geometry>
   </xacro:macro>
@@ -61,5 +65,5 @@
     <origin xyz="0 0 0" rpy="0 0 0" />
     <geometry>
-      <mesh filename="$(find sw_ros2_control_gazebo)/meshes/left_steering_hinge.STL" />
+      <mesh filename="$(find src_gazebo)/meshes/left_steering_hinge.STL" />
     </geometry>
   </xacro:macro>
@@ -67,5 +71,5 @@
     <origin xyz="0 0 0" rpy="0 0 0" />
     <geometry>
-      <mesh filename="$(find sw_ros2_control_gazebo)/meshes/right_steering_hinge.STL" />
+      <mesh filename="$(find src_gazebo)/meshes/right_steering_hinge.STL" />
     </geometry>
   </xacro:macro>

File: src_gazebo/urdf/src_ackermann.urdf (robot description, URDF)
Before this commit: robot src_ackermann, 14 links, 13 joints
Links:
- link chassis: geometry visual mesh filename=/home/kimsooyoung/ros2_ws/install/src_gazebo/share/src_gaze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
- link left_front_wheel: geometry collision cylinder length=0.045 radius=0.05; visual mesh filename=/home/kimsooyoung/ros2_ws/install/src_gazebo/share/src_gaze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
- link left_rear_wheel: geometry collision cylinder length=0.045 radius=0.05; visual mesh filename=/home/kimsooyoung/ros2_ws/install/src_gazebo/share/src_gaze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
- link left_steering_hinge: geometry visual mesh filename=/home/kimsooyoung/ros2_ws/install/src_gazebo/share/src_gaze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
- link right_front_wheel: geometry collision cylinder length=0.045 radius=0.05; visual mesh filename=/home/kimsooyoung/ros2_ws/install/src_gazebo/share/src_gaze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
- link right_rear_wheel: geometry collision cylinder length=0.045 radius=0.05; visual mesh filename=/home/kimsooyoung/ros2_ws/install/src_gazebo/share/src_gaze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
- link right_steering_hinge: geometry visual mesh filename=/home/kimsooyoung/ros2_ws/install/src_gazebo/share/src_gaze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
Joints:
- joint left_steering_hinge_joint: origin xyz=0.325 0.1 0 rpy=0 1.5708 0 -> xyz=0.325 0.1225 0 rpy=0 1.5708 0
- joint right_steering_hinge_joint: origin xyz=0.325 -0.1 0 rpy=0 1.5708 0 -> xyz=0.325 -0.1225 0 rpy=0 1.5708 0

File: src_gazebo/urdf/src_ackermann.urdf.xacro (robot description, xacro)
@@ -76,5 +76,6 @@
   </link>
   <joint name="left_steering_hinge_joint" type="revolute">
-    <origin xyz="0.325 0.1 0" rpy="0 1.5708 0" />
+    <!-- <origin xyz="0.325 0.1 0" rpy="0 1.5708 0" /> -->
+    <origin xyz="0.325 0.1225 0" rpy="0 1.5708 0" />
     <parent link="chassis" />
     <child link="left_steering_hinge" />
@@ -92,5 +93,6 @@
   </link>
   <joint name="right_steering_hinge_joint" type="continuous">
-    <origin xyz="0.325 -0.1 0" rpy="0 1.5708 0" />
+    <!-- <origin xyz="0.325 -0.100 0" rpy="0 1.5708 0" /> -->
+    <origin xyz="0.325 -0.1225 0" rpy="0 1.5708 0" />
     <parent link="chassis" />
     <child link="right_steering_hinge" />

Commit message: gz updated

File: src_gazebo/urdf/macros.xacro (robot description, xacro)
@@ -1,4 +1,4 @@
 <?xml version="1.0"?>
-<robot name="src_ackermann" xmlns:xacro="http://www.ros.org/wiki/xacro">
+<robot name="src_body" xmlns:xacro="http://www.ros.org/wiki/xacro">
   <!-- inertial parameter macros -->
   <xacro:macro name="chassis_inertial_params">
@@ -23,4 +23,10 @@
     <mass value="0.100" />
     <inertia ixx="4E-06" ixy="0" ixz="0" iyy="4E-06" iyz="0" izz="4E-06" />
+  </xacro:macro>
+  <xacro:macro name="steering_hinge_geometry">
+    <origin xyz="0 0 0" rpy="0 0 0" />
+    <geometry>
+      <box size="0.005 0.005 0.005"/>
+    </geometry>
   </xacro:macro>
   <xacro:macro name="hokuyo_inertial_params">
@@ -62,10 +68,4 @@
     </geometry>
   </xacro:macro>
-  <xacro:macro name="left_steering_hinge_geometry">
-    <origin xyz="0 0 0" rpy="0 0 0" />
-    <geometry>
-      <mesh filename="$(find src_gazebo)/meshes/left_steering_hinge.STL" />
-    </geometry>
-  </xacro:macro>
   <xacro:macro name="right_steering_hinge_geometry">
     <origin xyz="0 0 0" rpy="0 0 0" />
